Commit message: realsense collision test

File: src/ready2_educate/kuka_kr3_cell_description/urdf/cell.urdf.xacro (robot description, xacro)
@@ -107,4 +107,26 @@
             <child link="${prefix}camera"/>
         </joint>
+        <link name="${prefix}realsense_camera">
+            <visual>
+                <origin xyz="-0.0875 -0.052527 0.90" rpy="0 0 0"/>
+                <geometry>
+                    <box size="0.03 0.12 0.03"/>
+                </geometry>
+                <material name="red">
+                    <color rgba="0.9 0.5 0.5 1"/>
+                </material>
+            </visual>
+            <collision>
+                <origin xyz="-0.0875 -0.052527 0.90" rpy="0 0 0"/>
+                <geometry>
+                    <box size="0.03 0.12 0.03"/>
+                </geometry>
+            </collision>
+        </link>
+        <joint name="{prefix}realsense_camera_joint" type="fixed">
+            <origin xyz="-0.0325 0.264 0.7325" rpy="0 0 0"/>
+            <parent link="${prefix}cell_link"/>
+            <child link="${prefix}realsense_camera"/>
+        </joint>
     </xacro:macro>
 </robot>

Commit message: strange homepose

File: src/ready2_educate/kuka_kr3_cell_description/urdf/cell.urdf.xacro (robot description, xacro)
@@ -109,7 +109,7 @@
         <link name="${prefix}realsense_camera">
             <visual>
-                <origin xyz="-0.0875 -0.052527 0.90" rpy="0 0 0"/>
+                <origin xyz="-0.0875 -0.002527 0.9" rpy="0 0 0"/>
                 <geometry>
-                    <box size="0.03 0.12 0.03"/>
+                    <box size="0.12 0.04 0.04"/>
                 </geometry>
                 <material name="red">
@@ -118,7 +118,7 @@
             </visual>
             <collision>
-                <origin xyz="-0.0875 -0.052527 0.90" rpy="0 0 0"/>
+                <origin xyz="-0.0875 -0.002527 0.90" rpy="0 0 0"/>
                 <geometry>
-                    <box size="0.03 0.12 0.03"/>
+                    <box size="0.12 0.04 0.04"/>
                 </geometry>
             </collision>

Commit message: transformation

File: src/ready2_educate/kuka_kr3_cell_description/urdf/cell.urdf.xacro (robot description, xacro)
@@ -87,16 +87,16 @@
         <link name="${prefix}camera">
             <visual>
-                <origin xyz="-0.0875 -0.052527 0.995" rpy="0 0 0"/>
+                <origin xyz="-0.0575 -0.032527 1.01" rpy="0 0 0"/>
                 <geometry>
-                    <box size="0.045 0.053 0.195"/>
+                    <box size="0.09 0.09 0.225"/>
                 </geometry>
-                <material name="gray">
-                    <color rgba="0.5 0.5 0.5 1"/>
+                <material name="red">
+                    <color rgba="0.9 0.5 0.5 0.2"/>
                 </material>
             </visual>
             <collision>
-                <origin xyz="-0.0875 -0.052527 0.995" rpy="0 0 0"/>
+                <origin xyz="-0.0575 -0.032527 1.01" rpy="0 0 0"/>
                 <geometry>
-                    <box size="0.045 0.053 0.195"/>
+                    <box size="0.09 0.09 0.225"/>
                 </geometry>
             </collision>
@@ -109,16 +109,16 @@
         <link name="${prefix}realsense_camera">
             <visual>
-                <origin xyz="-0.0875 -0.002527 0.9" rpy="0 0 0"/>
+                <origin xyz="-0.0675 -0.002527 0.910" rpy="0 0 0"/>
                 <geometry>
-                    <box size="0.12 0.04 0.04"/>
+                    <box size="0.15 0.055 0.075"/>
                 </geometry>
                 <material name="red">
-                    <color rgba="0.9 0.5 0.5 1"/>
+                    <color rgba="0.9 0.5 0.5 0.2"/>
                 </material>
             </visual>
             <collision>
-                <origin xyz="-0.0875 -0.002527 0.90" rpy="0 0 0"/>
+                <origin xyz="-0.0675 -0.002527 0.910" rpy="0 0 0"/>
                 <geometry>
-                    <box size="0.12 0.04 0.04"/>
+                    <box size="0.15 0.055 0.075"/>
                 </geometry>
             </collision>
@@ -129,4 +129,20 @@
             <child link="${prefix}realsense_camera"/>
         </joint>
+        <link name="${prefix}realsense_camera_origin">
+            <visual>
+                    <origin xyz="0.0 -0.0 0.0" rpy="0 0 0"/>
+                    <geometry>
+                        <box size="0.01 0.01 0.01"/>
+                    </geometry>
+                    <material name="red">
+                        <color rgba="0.9 0.5 0.5 0.0"/>
+                    </material>
+                </visual>
+        </link>
+        <joint name="{prefix}realsense_camera_origin_joint" type="fixed">
+            <origin xyz="-0.068 0.260 1.661" rpy="0 3.14159265359 0"/>
+            <parent link="${prefix}cell_link"/>
+            <child link="${prefix}realsense_camera_origin"/>
+        </joint>
     </xacro:macro>
 </robot>

Commit message: sebbi sehr glüglich

File: src/ready2_educate/kuka_kr3_cell_description/urdf/cell.urdf.xacro (robot description, xacro)
@@ -141,5 +141,5 @@
         </link>
         <joint name="{prefix}realsense_camera_origin_joint" type="fixed">
-            <origin xyz="-0.068 0.260 1.661" rpy="0 3.14159265359 0"/>
+            <origin xyz="-0.068 0.260 1.661" rpy="0 0 0"/> <!--<origin xyz="-0.068 0.260 1.661" rpy="0 3.14159265359 0"/>-->
             <parent link="${prefix}cell_link"/>
             <child link="${prefix}realsense_camera_origin"/>
